File: Harware/ATMega128_Breakout.sch (KiCad schematic (older format))
At the start: 22 parts, among them IC1 ATMEGA128-A, J1 SIL8, J2 SIL8, P1 CONN_10, P2 CONN_10, P3 CONN_10, P4 CONN_10, P5 CONN_2, P8 CONN_5X2, SW1 rst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

Commit message: changed design
Parts:
- removed D3, D4: LED, ~, symbol LED
- removed P5: CONN_2, symbol CONN_2
- removed R3: 470r, ~, symbol R
- added JP1: JUMPER, ~, symbol JUMPER
- added P6: CONN_7, symbol CONN_7
Connections:
- net +5V: now also P6.3 (P3)
- net GND: now also P6.1 (P1)
- net RST: now also JP1.1
- net RX0: now also P6.4 (P4)
- net TX0: now also P6.5 (P5)
- net INTR: now reaches IC1.25 ((SCL/INT0)PD0), P2.3 (P3)
- net INTR: now also P4.9 (P9)
- net RX1: no longer names the net of IC1.27 ((RXD1/INT2)PD2), P2.5 (P5)
- net TX1: no longer names the net of IC1.28 ((TXD1/INT3)PD3), P2.6 (P6)
- new net: JP1.2, P6.7 (P7)
- no-connect marks 12 -> 13
Changed lines of the file:
@@
 Sheet 1 1
 Title ""
-Date "22 may 2015"
+Date "30 may 2015"
 Rev ""
 Comp "ExploreEmbedded.com"
@@
 	1    0    0    -1
 $EndComp
-$Comp
-L ATMEGA128-A IC1
-U 1 1 5553099A
-P 5700 3000
-F 0 "IC1" H 4600 4850 50  0000 L BNN
-F 1 "ATMEGA128-A" H 6250 1100 50  0000 L BNN
-F 2 "TQFP64" H 4750 1150 50  0001 C CNN
-F 3 "" H 5700 3000 60  0001 C CNN
-	1    5700 3000
-	1    0    0    -1
-$EndComp
 Text Label 9950 2900 2    60   ~ 0
 RST
@@
 Wire Wire Line
 	7400 3100 7000 3100
-Text Label 8700 4250 2    40   ~ 0
-TX1
-Text Label 8700 4450 2    40   ~ 0
-RX1
 Text Label 4400 4000 2    40   ~ 0
 RX0
@@
 Text Label 1550 1100 2    40   ~ 0
 TX0
-$Comp
-L LED D3
-U 1 1 55544658
-P 1950 1300
-F 0 "D3" H 1950 1400 50  0000 C CNN
-F 1 "LED" H 1950 1200 50  0000 C CNN
-F 2 "~" H 1950 1300 60  0000 C CNN
-F 3 "~" H 1950 1300 60  0000 C CNN
-	1    1950 1300
-	0    1    1    0
-$EndComp
-$Comp
-L LED D4
-U 1 1 5554465E
-P 2350 1300
-F 0 "D4" H 2350 1400 50  0000 C CNN
-F 1 "LED" H 2350 1200 50  0000 C CNN
-F 2 "~" H 2350 1300 60  0000 C CNN
-F 3 "~" H 2350 1300 60  0000 C CNN
-	1    2350 1300
-	0    1    1    0
-$EndComp
-$Comp
-L R R3
-U 1 1 55544664
-P 2350 1850
-F 0 "R3" V 2430 1850 40  0000 C CNN
-F 1 "470r" V 2357 1851 40  0000 C CNN
-F 2 "~" V 2280 1850 30  0000 C CNN
-F 3 "~" H 2350 1850 30  0000 C CNN
-	1    2350 1850
-	1    0    0    -1
-$EndComp
-$Comp
-L GND #PWR08
-U 1 1 5554466A
-P 2350 2150
-F 0 "#PWR08" H 2350 2150 30  0001 C CNN
-F 1 "GND" H 2350 2080 30  0001 C CNN
-F 2 "" H 2350 2150 60  0001 C CNN
-F 3 "" H 2350 2150 60  0001 C CNN
-	1    2350 2150
-	1    0    0    -1
-$EndComp
-Wire Wire Line
-	1950 1500 2350 1500
-Wire Wire Line
-	2350 1500 2350 1600
-Text Label 7000 4300 0    40   ~ 0
-TX1
-Text Label 7000 4200 0    40   ~ 0
-RX1
 NoConn ~ 4400 2700
 NoConn ~ 4400 2800
 NoConn ~ 4400 2900
-Text Label 1950 1100 2    40   ~ 0
-RX1
-Text Label 2350 1100 2    40   ~ 0
-TX1
-Wire Wire Line
-	2350 2100 2350 2150
 Text Label 9950 3100 2    40   ~ 0
 TX0
 NoConn ~ 4400 2500
 NoConn ~ 4400 2600
-$Comp
-L CONN_2 P5
-U 1 1 555D6E6F
-P 9050 4350
-F 0 "P5" V 9000 4350 40  0000 C CNN
-F 1 "CONN_2" V 9100 4350 40  0000 C CNN
-F 2 "" H 9050 4350 60  0000 C CNN
-F 3 "" H 9050 4350 60  0000 C CNN
-	1    9050 4350
-	1    0    0    -1
-$EndComp
-NoConn ~ 8700 3800
-NoConn ~ 8700 3900
 Wire Notes Line
 	500  5200 11200 5200
@@
 EndData
 $EndBitmap
+$Comp
+L CONN_7 P6
+U 1 1 5569E83B
+P 10950 1400
+F 0 "P6" V 10920 1400 60  0000 C CNN
+F 1 "CONN_7" V 11020 1400 60  0000 C CNN
+F 2 "" H 10950 1400 60  0000 C CNN
+F 3 "" H 10950 1400 60  0000 C CNN
+	1    10950 1400
+	1    0    0    -1
+$EndComp
+Text Label 10600 1400 2    40   ~ 0
+RX0
+Text Label 10600 1500 2    40   ~ 0
+TX0
+$Comp
+L JUMPER JP1
+U 1 1 5569EB29
+P 10150 1700
+F 0 "JP1" H 10150 1850 60  0000 C CNN
+F 1 "JUMPER" H 10150 1620 40  0000 C CNN
+F 2 "~" H 10150 1700 60  0000 C CNN
+F 3 "~" H 10150 1700 60  0000 C CNN
+	1    10150 1700
+	1    0    0    -1
+$EndComp
+Wire Wire Line
+	10600 1700 10450 1700
+Text Label 9850 1700 2    60   ~ 0
+RST
+Text Label 10600 1300 2    60   ~ 0
++5V
+$Comp
+L GND #PWR08
+U 1 1 5569ECBD
+P 10250 1200
+F 0 "#PWR08" H 10250 1200 30  0001 C CNN
+F 1 "GND" H 10250 1130 30  0001 C CNN
+F 2 "" H 10250 1200 60  0001 C CNN
+F 3 "" H 10250 1200 60  0001 C CNN
+	1    10250 1200
+	1    0    0    -1
+$EndComp
+Wire Wire Line
+	10250 1200 10250 1100
+Wire Wire Line
+	10250 1100 10600 1100
+NoConn ~ 10600 1200
+NoConn ~ 10600 1600
+Text Label 7000 4000 0    60   ~ 0
+INTR
+Text Label 8700 3800 2    60   ~ 0
+INTR
+$Comp
+L ATMEGA128-A IC1
+U 1 1 5553099A
+P 5700 3000
+F 0 "IC1" H 4600 4850 50  0000 L BNN
+F 1 "ATMEGA128-A" H 6250 1100 50  0000 L BNN
+F 2 "TQFP64" H 4750 1150 50  0001 C CNN
+F 3 "" H 5700 3000 60  0001 C CNN
+	1    5700 3000
+	1    0    0    -1
+$EndComp
+NoConn ~ 8700 3900
 $EndSCHEMATC

Commit message: added final files
Parts:
- added D3: LED, ~, symbol LED
- added R3: 470r, ~, symbol R
Connections:
- net +5V: now also R3.1
- net GND: now also D3.2 (K)
- new net: D3.1 (A), R3.2
Changed lines of the file:
@@
 LIBS:at128-cache
 LIBS:ATMega128_Breakout-cache
-EELAYER 27 0
+EELAYER 25 0
 EELAYER END
 $Descr A4 11693 8268
@@
 $EndDescr
 $Comp
-L GND #PWR01
+L GND #PWR4
 U 1 1 555308F4
 P 3150 2000
-F 0 "#PWR01" H 3150 2000 30  0001 C CNN
+F 0 "#PWR4" H 3150 2000 30  0001 C CNN
 F 1 "GND" H 3150 1930 30  0001 C CNN
 F 2 "" H 3150 2000 60  0001 C CNN
@@
 $EndComp
 $Comp
-L GND #PWR02
+L GND #PWR2
 U 1 1 55530913
 P 1950 4150
-F 0 "#PWR02" H 1950 4150 30  0001 C CNN
+F 0 "#PWR2" H 1950 4150 30  0001 C CNN
 F 1 "GND" H 1950 4080 30  0001 C CNN
 F 2 "" H 1950 4150 60  0001 C CNN
@@
 $EndComp
 $Comp
-L GND #PWR03
+L GND #PWR9
 U 1 1 5553095B
 P 10750 3200
-F 0 "#PWR03" H 10750 3200 30  0001 C CNN
+F 0 "#PWR9" H 10750 3200 30  0001 C CNN
 F 1 "GND" H 10750 3130 30  0001 C CNN
 F 2 "" H 10750 3200 60  0001 C CNN
@@
 $EndComp
 $Comp
-L GND #PWR04
+L GND #PWR6
 U 1 1 55530961
 P 6800 950
-F 0 "#PWR04" H 6800 950 30  0001 C CNN
+F 0 "#PWR6" H 6800 950 30  0001 C CNN
 F 1 "GND" H 6800 880 30  0001 C CNN
 F 2 "" H 6800 950 60  0001 C CNN
@@
 $EndComp
 $Comp
-L GND #PWR05
+L GND #PWR5
 U 1 1 55530994
 P 5650 5050
-F 0 "#PWR05" H 5650 5050 30  0001 C CNN
+F 0 "#PWR5" H 5650 5050 30  0001 C CNN
 F 1 "GND" H 5650 4980 30  0001 C CNN
 F 2 "" H 5650 5050 60  0001 C CNN
@@
 	7450 1300 7000 1300
 $Comp
-L GND #PWR06
+L GND #PWR7
 U 1 1 55535CD2
 P 8350 1150
-F 0 "#PWR06" H 8350 1150 30  0001 C CNN
+F 0 "#PWR7" H 8350 1150 30  0001 C CNN
 F 1 "GND" H 8350 1080 30  0001 C CNN
 F 2 "" H 8350 1150 60  0001 C CNN
@@
 	1150 1500 1150 1600
 $Comp
-L GND #PWR07
+L GND #PWR1
 U 1 1 555361A0
 P 1150 2150
-F 0 "#PWR07" H 1150 2150 30  0001 C CNN
+F 0 "#PWR1" H 1150 2150 30  0001 C CNN
 F 1 "GND" H 1150 2080 30  0001 C CNN
 F 2 "" H 1150 2150 60  0001 C CNN
@@
 43 7C 02 00 00 84 0C F1 09 00 00 10 32 C4 27 00 00 40 C8 10 9F 00 00 00 21 43 7C 02 00 00 84 0C
 F1 09 00 00 10 32 C4 27 00 00 40 C8 10 9F 00 00 00 21 43 7C 02 00 00 84 EC FF 02 24 05 F2 19 03
-C8 1D 6B 00 00 00 00 49 45 4E 44 AE 42 60 82 00 $EndBitmap
+C8 1D 6B 00 00 00 00 49 45 4E 44 AE 42 60 82 00
 EndData
 $EndBitmap
@@
 +5V
 $Comp
-L GND #PWR08
+L GND #PWR8
 U 1 1 5569ECBD
 P 10250 1200
-F 0 "#PWR08" H 10250 1200 30  0001 C CNN
+F 0 "#PWR8" H 10250 1200 30  0001 C CNN
 F 1 "GND" H 10250 1130 30  0001 C CNN
 F 2 "" H 10250 1200 60  0001 C CNN
@@
 $EndComp
 NoConn ~ 8700 3900
+$Comp
+L R R3
+U 1 1 558108C2
+P 2500 1250
+F 0 "R3" V 2580 1250 40  0000 C CNN
+F 1 "470r" V 2507 1251 40  0000 C CNN
+F 2 "~" V 2430 1250 30  0000 C CNN
+F 3 "~" H 2500 1250 30  0000 C CNN
+	1    2500 1250
+	1    0    0    -1
+$EndComp
+$Comp
+L LED D3
+U 1 1 5581091F
+P 2500 1800
+F 0 "D3" H 2500 1900 50  0000 C CNN
+F 1 "LED" H 2500 1700 50  0000 C CNN
+F 2 "~" H 2500 1800 60  0000 C CNN
+F 3 "~" H 2500 1800 60  0000 C CNN
+	1    2500 1800
+	0    1    1    0
+$EndComp
+Wire Wire Line
+	2500 1500 2500 1600
+$Comp
+L GND #PWR3
+U 1 1 558109FA
+P 2500 2100
+F 0 "#PWR3" H 2500 2100 30  0001 C CNN
+F 1 "GND" H 2500 2030 30  0001 C CNN
+F 2 "" H 2500 2100 60  0001 C CNN
+F 3 "" H 2500 2100 60  0001 C CNN
+	1    2500 2100
+	1    0    0    -1
+$EndComp
+Wire Wire Line
+	2500 2000 2500 2100
+Text Label 2500 1000 0    60   ~ 0
++5V
 $EndSCHEMATC
