File: Harware/ATMega128_Breakout.kicad_pcb (KiCad board)
At the start: 2 copper layers, 40.6 x 73.7 mm, 22 parts, among them IC1 ATMEGA128-A, J1 SIL8, J2 SIL8, P1 CONN_10, P2 CONN_10, P3 CONN_10, P4 CONN_10, P5 CONN_2, P8 CONN_5X2, SW1 rst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

Commit message: changed design
Parts:
- removed D3, D4: LED, SM1206
- removed P5: CONN_2, SIL-2
- removed R3: 470r, SM1206
- added JP1: JUMPER, SIL-2, F.Cu at (95.8, 105.9)
- added P6: CONN_7, SIL-7, F.Cu at (78.7, 105.2)
- moved P8 122.1 mm to (78.2, 50.3)
- moved J2 99.6 mm to (67.8, 39.4)
- moved J1 99.6 mm to (88.1, 39.4)
- moved C3 99.3 mm to (78.6, 76.1)
- moved SW1 99.3 mm to (62.7, 106.9)
- moved C1 99.3 mm to (85.6, 89.2)
- moved C4 99.3 mm to (81.0, 73.7)
- moved IC1 99.3 mm to (78.0, 73.9)
- moved P3 99.3 mm to (95.8, 63.8)
- moved P4 99.3 mm to (95.8, 89.2)
- moved R1 99.3 mm to (71.6, 98.0)
- moved X1 99.3 mm to (78.0, 89.2)
- moved C2 99.3 mm to (70.4, 89.2)
- moved P1 99.3 mm to (60.2, 63.8)
- moved P2 99.3 mm to (60.2, 89.2)
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Connections:
- net /RX1 renamed N-0000036
- net /TX1 renamed N-0000034
- IC1 pad 25: N-0000016 (its old number) -> /INTR
- P2 pad 3: N-0000016 (its old number) -> /INTR
- P4 pad 9: (no net) -> /INTR
Routing:
- net N-0000034: track 155.7 -> 17.8 mm, vias 2 -> 0
- net N-0000036: track 148.4 -> 16.4 mm, vias 1 -> 0
- net /RST: track 61.9 -> 149.9 mm, vias 1 -> 3
- net GND: track 276.1 -> 232.0 mm, vias 5 -> 4
- net /SCK: track 82.1 -> 40.3 mm, vias 1 -> 0
- net /INTR: track 0.00 -> 41.7 mm, vias 0 -> 2
- net /TX0: track 130.5 -> 156.9 mm, vias 2 -> 1
- net N-0000031 (its old number): track 18.3 -> 0.00 mm, vias 2 -> 0
- net N-0000016 (its old number): track 14.9 -> 0.00 mm
- net /RX0: track 158.8 -> 171.5 mm, vias 2 -> 0
- net N-0000042: track 0.00 -> 9.61 mm
- net N-0000045: track 27.8 -> 33.1 mm
- net N-0000041: track 26.8 -> 32.1 mm
- net N-0000048: track 27.7 -> 31.9 mm
- net N-0000013: track 14.7 -> 11.6 mm, vias 2 -> 1
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- added copper zone on F.Cu, net /+5V
- added copper zone on B.Cu, net GND
Other:
- board size 40.6 x 73.7 mm -> 40.5 x 75.1 mm
- board text added: "5V"
- board text added: "Boot Jumper"
- board text added: "COMP"
- board text added: "DTR"
- board text added: "Explore ATMega-128"
- board text added: "INTR"
- board text added: "RX"
- board text added: "SOLD"
- board text added: "TX"
- board text removed: "ATMega-128"
- board text removed: "RX1"
- board text removed: "TX1"

Commit message: added final files
Parts:
- added D3: LED, ex:LED-1206_NEW, F.Cu at (94.9, 45.2)
- added LOGO: , EE:LOGO (2), B.Cu at (83.0, 56.5)
- added R3: 470r, SM1206, B.Cu at (94.9, 48.8)
- D1, D2: footprint SM1206 -> ex:LED-1206_NEW
- P8: footprint VASCH5x2 -> Connect:VASCH5x2
- X1: footprint HC-49V -> Discret:HC-49V
Connections:
- IC1 pad 1: (no net) -> Net-(IC1-Pad1)
- IC1 pad 18: (no net) -> Net-(IC1-Pad18)
- IC1 pad 19: (no net) -> Net-(IC1-Pad19)
- IC1 pad 33: (no net) -> Net-(IC1-Pad33)
- IC1 pad 34: (no net) -> Net-(IC1-Pad34)
- IC1 pad 43: (no net) -> Net-(IC1-Pad43)
- P2 pad 2: (no net) -> Net-(P2-Pad2)
- P4 pad 10: (no net) -> Net-(P4-Pad10)
- P6 pad 2: (no net) -> Net-(P6-Pad2)
- P6 pad 6: (no net) -> Net-(P6-Pad6)
- P8 pad 3: (no net) -> Net-(P8-Pad3)
- P8 pad 4: (no net) -> Net-(P8-Pad4)
- P8 pad 6: (no net) -> Net-(P8-Pad6)
Routing:
- net GND: track 232.0 -> 248.9 mm, vias 4 -> 5
- net /RST: track 149.9 -> 159.6 mm
- net /+5V: track 117.8 -> 123.7 mm
- net Net-(IC1-Pad54): track 35.3 -> 40.7 mm
- net Net-(D3-Pad1): track 0.00 -> 3.87 mm, vias 0 -> 1
Other:
- board size 40.5 x 75.1 mm -> 41 x 75 mm
- board text added: "(SCL/INTR0)"
- board text added: "(SDA/INTR1)"
- board text added: "Explore ATMega128 Breakout"
- board text added: "ExploreEmbedded.com"
- board text added: "PB4 *"
- board text added: "PB5 *"
- board text added: "PB6 *"
- board text added: "PB7 *"
- board text added: "PD2(RX1)"
- board text added: "PD3(TX1)"
- board text added: "PE3 *"
- board text added: "PE4 *"
- board text added: "PE5 *"
- board text removed: "Explore ATMega-128"
- board text removed: "PB4"
- board text removed: "PB5"
- board text removed: "PB6"
- board text removed: "PB7"
- board text removed: "PD2"
- board text removed: "PD3"
- board text removed: "PE3"
- board text removed: "PE4"
- board text removed: "PE5"

Commit message: k
Parts:
- SW1: value rst -> RESET
- moved LOGO 12.0 mm to (71.6, 52.6), turned to 270 degrees
Other:
- board text added: "Boot"
- board text added: "Explore ATMega128"
- board text removed: "Boot Jumper"
- board text removed: "Explore ATMega128 Breakout"
